File: switch_main_v4/1000base-t1-phy-1.kicad_sch (KiCad schematic)
At the start: 39 parts, among them Q1401 DMN21D2UFB-7B, Q1402 DMP21D0UFB-7B, U1401 TPS62290TDRVRQ1, U1402 88Q2112-A2-NYD2A000-P123

Commit message: Fixed mistake where RMII TX and RX signals were swapped
Parts:
- removed R1410: 4k7, Resistor_SMD:R_0402_1005Metric, symbol Device:R_Small
- R1401: now fitted; now in the parts list
Connections:
- net RX_CTL: now also R1401.2
- net RX_D1: no longer R1401.2
Other:
- moved on the sheet: R1403
