File: switch_main_v4/primary-mcu.kicad_sch (KiCad schematic)
At the start: 51 parts, among them Q801 DMP21D0UFB-7B, U801 FM25CL64B-DG, U802 STM32H573IIKxQ, Y801 XRCGB25M000F2P02R0, Y802 ECS-.327-7-12QS-TR

Commit message: Fixed mistake where RMII TX and RX signals were swapped
Parts:
- Y801: value XRCGB25M000F2P02R0 -> XRCGB25M000F3A16R0; footprint project_footprints:NX2016SA-40M-STD-CZS-3 -> project_footprints:XRCGB25M000F3A16R0
Changed lines of the file:
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@@
 			)
 		)
-		(property "Value" "XRCGB25M000F2P02R0"
+		(property "Value" "XRCGB25M000F3A16R0"
 			(at 66.04 208.28 90)
 			(effects
@@
 			)
 		)
-		(property "Footprint" "project_footprints:NX2016SA-40M-STD-CZS-3"
+		(property "Footprint" "project_footprints:XRCGB25M000F3A16R0"
 			(at 99.06 208.28 0)
 			(effects
