File: switch_main_v4/switch.kicad_sch (KiCad schematic)
At the start: 43 parts, among them U901 SJA1105QELY, Y901 XRCGB25M000F2P02R0

Commit message: Fixed mistake where RMII TX and RX signals were swapped
Parts:
- Y901: value XRCGB25M000F2P02R0 -> XRCGB25M000F3A16R0
Connections:
- net xMII4.RX_ER is gone; now on net GND1: U901.P13 (MII4_RX_ER)
- net xMII4.RX_CRS_DV: now also U901.P9 (MII4_TX_EN/TX_CTL); no longer U901.N12 (MII4_RX_DV/CRS_DV/RX_CTL)
- net xMII4.RX_D0: now also U901.P7 (MII4_TXD0); no longer U901.N10 (MII4_RXD0)
- net xMII4.RX_D1: now also U901.N7 (MII4_TXD1); no longer U901.P11 (MII4_RXD1)
- net xMII4.TX_D0: now also U901.N10 (MII4_RXD0); no longer U901.P7 (MII4_TXD0)
- net xMII4.TX_D1: now also U901.P11 (MII4_RXD1); no longer U901.N7 (MII4_TXD1)
- net xMII4.TX_EN: now also U901.N12 (MII4_RX_DV/CRS_DV/RX_CTL); no longer U901.P9 (MII4_TX_EN/TX_CTL)
Changed lines of the file:
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@@
 	)
 	(junction
+		(at 254 88.9)
+		(diameter 0)
+		(color 0 0 0 0)
+	)
+	(junction
 		(at 116.84 111.76)
 		(diameter 0)
@@
 	)
 	(bus_entry
-		(at 228.6 86.36)
-		(size 2.54 2.54)
-		(stroke
-			(width 0)
-			(type default)
-		)
-	)
-	(bus_entry
 		(at 360.68 78.74)
 		(size -2.54 2.54)
@@
 	(wire
 		(pts
+			(xy 254 88.9) (xy 256.54 88.9)
+		)
+		(stroke
+			(width 0)
+			(type default)
+		)
+	)
+	(wire
+		(pts
 			(xy 78.74 53.34) (xy 88.9 53.34)
 		)
@@
 		)
 	)
+	(wire
+		(pts
+			(xy 254 88.9) (xy 254 91.44)
+		)
+		(stroke
+			(width 0)
+			(type default)
+		)
+	)
 	(bus
 		(pts
@@
 	(wire
 		(pts
-			(xy 256.54 88.9) (xy 231.14 88.9)
-		)
-		(stroke
-			(width 0)
-			(type default)
-		)
-	)
-	(wire
-		(pts
 			(xy 48.26 256.54) (xy 48.26 259.08)
 		)
@@
 		)
 	)
-	(bus
-		(pts
-			(xy 228.6 86.36) (xy 228.6 81.28)
-		)
-		(stroke
-			(width 0)
-			(type default)
-		)
-	)
 	(wire
 		(pts
@@
 	(wire
 		(pts
-			(xy 254 86.36) (xy 254 91.44)
+			(xy 254 86.36) (xy 254 88.9)
 		)
 		(stroke
@@
 	)
 	(label "xMII4.TX_D1"
-		(at 251.46 55.88 180)
+		(at 251.46 76.2 180)
 		(effects
 			(font
@@
 	)
 	(label "xMII4.TX_EN"
-		(at 251.46 63.5 180)
+		(at 251.46 83.82 180)
 		(effects
 			(font
@@
 	)
 	(label "xMII4.RX_D1"
-		(at 251.46 76.2 180)
+		(at 251.46 55.88 180)
 		(effects
 			(font
@@
 	)
 	(label "xMII4.RX_CRS_DV"
-		(at 251.46 83.82 180)
+		(at 251.46 63.5 180)
 		(effects
 			(font
@@
 	)
 	(label "xMII4.RX_D0"
-		(at 251.46 73.66 180)
+		(at 251.46 53.34 180)
 		(effects
 			(font
@@
 	)
 	(label "xMII4.TX_D0"
-		(at 251.46 53.34 180)
-		(effects
-			(font
-				(size 1.27 1.27)
-			)
-			(justify right bottom)
-		)
-	)
-	(label "xMII4.RX_ER"
-		(at 251.46 88.9 180)
+		(at 251.46 73.66 180)
 		(effects
 			(font
@@
 			)
 		)
-		(property "Value" "XRCGB25M000F2P02R0"
+		(property "Value" "XRCGB25M000F3A16R0"
 			(at 205.74 162.56 90)
 			(effects
