File: switch_main_v4/power-in-isolated.kicad_sch (KiCad schematic)
At the start: 13 parts, among them J601 MKXS1-1 Power Input, U601 TVS3301DRBR, U602 TPS26600RHFR

Commit message: Updated power connector model
Parts:
- J601: footprint project_footprints:10132798-031100LF -> project_footprints:10132797-031100LF
Changed lines of the file:
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@@
 			)
 		)
-		(property "Footprint" "project_footprints:10132798-031100LF"
+		(property "Footprint" "project_footprints:10132797-031100LF"
 			(at 27.94 88.9 0)
 			(effects
