File: switch_main_v4/power-in.kicad_sch (KiCad schematic)
At the start: 13 parts, among them J301 MKXS1-1 Power Input, U301 TVS3301DRBR, U302 TPS26600RHFR

Commit message: Updated power connector model
Parts:
- J301: footprint project_footprints:10132798-031100LF -> project_footprints:10132797-031100LF
Changed lines of the file:
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@@
 			)
 		)
-		(property "Footprint" "project_footprints:10132798-031100LF"
+		(property "Footprint" "project_footprints:10132797-031100LF"
 			(at 43.18 88.9 0)
 			(effects
