File: switch_main_v4/switch_main_v4.kicad_pcb (KiCad board)
At the start: 6 copper layers, 65 x 50 mm, 471 parts, among them J2401 JST-GH-2-Horizontal, J2402 JST-GH-2-Horizontal, J2403 MSPE-J2L0-B00, J2404 MSPE-J2L0-B00, J2405 MSPE-J2L0-x00, J301 MKXS1-1 Power Input, J601 MKXS1-1 Power Input, Q1101 DMN21D2UFB-7B, Q1102 DMN21D2UFB-7B, Q1103 DMN21D2UFB-7B, Q1301 DMN21D2UFB-7B, Q1302 DMP21D0UFB-7B, Q1401 DMN21D2UFB-7B, Q1402 DMP21D0UFB-7B, Q1501 DMN21D2UFB-7B, Q1502 DMP21D0UFB-7B, Q2201 DMP21D0UFB-7B, Q2202 DMP21D0UFB-7B, Q2203 DMN21D2UFB-7B, Q2204 DMP21D0UFB-7B, Q2205 DMN21D2UFB-7B, Q2206 DMP21D0UFB-7B, Q2301 DMN21D2UFB-7B, Q2302 DMP21D0UFB-7B, Q2601 DMN21D2UFB-7B, Q2602 DMN21D2UFB-7B, Q801 DMP21D0UFB-7B, T1801 74930100, T1901 74930100, T2001 74930100, T2101 74930100, U1201 LMK1C1104DQFR, U1301 TPS62290TDRVRQ1, U1302 88Q2112-A2-NYD2A000-P123, U1401 TPS62290TDRVRQ1, U1402 88Q2112-A2-NYD2A000-P123, U1501 TPS62290TDRVRQ1, U1502 88Q2112-A2-NYD2A000-P123, U1601 LAN8671C2-E_U3B, U2201 TPS27S100BRRK, U2202 TPS27S100BRRK, U2301 NCS213RMUTAG, U2302 TPS27S100BRRK, U2501 ISO6521REUR, U2502 ISO6520REUR, U2601 STM32H503KBUx, U301 TVS3301DRBR, U302 TPS26600RHFR, U401 TPS7B8133QDRVRQ1, U402 LMQ66420MC3RXBRQ1, U403 TPS2116DRL, U501 TPS62290TDRVRQ1, U502 TPS62290TDRVRQ1, U601 TVS3301DRBR, U602 TPS26600RHFR, U701 TPS7B8133QDRVRQ1, U702 MAX20075DATCA/V+, U703 NCP508MT25TBG, U801 FM25CL64B-DG, U802 STM32H573IIKxQ, U901 SJA1105QELY, Y801 XRCGB25M000F2P02R0, Y802 ECS-.327-7-12QS-TR, Y901 XRCGB25M000F2P02R0

Commit message: Updated power connector model
Parts:
- J301, J601: footprint project_footprints:10132798-031100LF -> project_footprints:10132797-031100LF
- Y801: value XRCGB25M000F2P02R0 -> XRCGB25M000F3A16R0; footprint project_footprints:NX2016SA-40M-STD-CZS-3 -> project_footprints:XRCGB25M000F3A16R0
- Y901: value XRCGB25M000F2P02R0 -> XRCGB25M000F3A16R0
- turned J301 to -90 degrees
- turned J601 to -90 degrees
