File: pcbs/switch-main-v4/1000base-t1-phy-0.kicad_sch (KiCad schematic)
At the start: 38 parts, among them Q1301 DMN21D2UFB-7B, Q1302 DMP21D0UFB-7B, U1301 TPS62290TDRVRQ1, U1302 88Q2112-A2-NYD2A000-P123

Commit message: Updated to Kicad v10
Parts:
- C1322, R1302, R1304: now left out of the parts list
