File: pcbs/switch-main-v4/1000base-t1-phy-1.kicad_sch (KiCad schematic)
At the start: 38 parts, among them Q1401 DMN21D2UFB-7B, Q1402 DMP21D0UFB-7B, U1401 TPS62290TDRVRQ1, U1402 88Q2112-A2-NYD2A000-P123

Commit message: Updated to Kicad v10
Parts:
- C1422, R1402, R1404: now left out of the parts list
