File: pcbs/switch-main-v4/1000base-t1-phy-2.kicad_sch (KiCad schematic)
At the start: 38 parts, among them Q1501 DMN21D2UFB-7B, Q1502 DMP21D0UFB-7B, U1501 TPS62290TDRVRQ1, U1502 88Q2112-A2-NYD2A000-P123

Commit message: Updated to Kicad v10
Parts:
- C1522, R1502, R1504: now left out of the parts list
