File: pcbs/switch-main-v4/10base-t1s-phy.kicad_sch (KiCad schematic)
At the start: 20 parts, among them U1601 LAN8671C2-E_U3B

Commit message: Updated to Kicad v10
Parts:
- R1603: now left out of the parts list
